File: KiCad/dadboard.kicad_pcb (KiCad board)
At the start: 2 copper layers, 397 x 162 mm, 258 parts, among them SW1 Rotary_Encoder_Switch, U1 ATmega32U4-AU, U2 ATmega32U4-AU

Commit message: Finished matrix
Parts:
- removed the REF** at (225.9, -59.6)
- removed the REF** at (-24.3, -59.6)
- removed the REF** at (232.3, -59.6)
- removed the REF** at (-17.9, -59.6)
- added C1: 22pF, Footprints:C_0805_2012Metric, B.Cu at (-62.7, -30.1)
- added C10: .1uF, Footprints:C_0805_2012Metric, B.Cu at (274.1, -146.2)
- added C11: .1uF, Footprints:C_0805_2012Metric, B.Cu at (349.3, -201.7)
- added C12: 10uF, Footprints:C_0805_2012Metric, B.Cu at (283.2, -140.3)
- added C13: .1uF, Footprints:C_0805_2012Metric, B.Cu at (278.5, -146.2)
- added C14: .1uF, Footprints:C_0805_2012Metric, B.Cu at (344.8, -201.7)
- added C15: .1uF, Footprints:C_0805_2012Metric, B.Cu at (344.8, -195.8)
- added C16: .1uF, Footprints:C_0805_2012Metric, B.Cu at (353.7, -204.7)
- added C2: 22pF, Footprints:C_0805_2012Metric, B.Cu at (283.2, -149.1)
- added C3: 22pF, Footprints:C_0805_2012Metric, B.Cu at (-57.1, -35.7)
- added C4: 22pF, Footprints:C_0805_2012Metric, B.Cu at (349.3, -195.8)
- added C5: 1uF, Footprints:C_0805_2012Metric, B.Cu at (278.8, -149.1)
- added C6: 1uF, Footprints:C_0805_2012Metric, B.Cu at (344.8, -204.7)
- added C7: 10uF, Footprints:C_0805_2012Metric, B.Cu at (287.3, -143.2)
- added C8: .1uF, Footprints:C_0805_2012Metric, B.Cu at (349.3, -198.8)
- added C9: .1uF, Footprints:C_0805_2012Metric, B.Cu at (344.8, -198.8)
- added F1: Polyfuse_Small, Footprints:Fuse_0805_2012Metric, B.Cu at (353.7, -201.7)
- added F2: Polyfuse_Small, Footprints:Fuse_0805_2012Metric, B.Cu at (349.3, -204.7)
- added JP1: Jumper, Footprints:ResetJumper, F.Cu at (274.2, -139.3)
- added JP2: Jumper, Footprints:ResetJumper, F.Cu at (265.9, -139.3)
- added MX101: K, MX_Only:MXOnly-1U-NoLED, F.Cu at (151.7, 11.9)
- added MX103: L, MX_Only:MXOnly-1U-NoLED, F.Cu at (170.8, 11.9)
- added MX105: ;, MX_Only:MXOnly-1U-NoLED, F.Cu at (189.8, 11.9)
- added MX108: ', MX_Only:MXOnly-1U-Hotswap, F.Cu at (208.9, 11.9)
- added MX11: F8, MX_Only:MXOnly-1U-Hotswap, F.Cu at (146.9, -50.0)
- added MX110: Enter, MX_Only:MXOnly-2.25U-Hotswap, F.Cu at (239.8, 11.9)
- added MX111: Pg Dn, MX_Only:MXOnly-1U-NoLED, F.Cu at (280.3, 11.9)
- added MX13: F9, MX_Only:MXOnly-1U-Hotswap, F.Cu at (170.8, -50.0)
- added MX130: N, MX_Only:MXOnly-1U-NoLED, F.Cu at (123.1, 31.0)
- added MX133: M, MX_Only:MXOnly-1U-Hotswap, F.Cu at (142.2, 31.0)
- added MX134: ,, MX_Only:MXOnly-1U-NoLED, F.Cu at (161.2, 31.0)
- added MX137: ., MX_Only:MXOnly-1U-Hotswap, F.Cu at (180.3, 31.0)
- added MX139: /, MX_Only:MXOnly-1U-Hotswap, F.Cu at (199.3, 31.0)
- added MX14: F10, MX_Only:MXOnly-1U-NoLED, F.Cu at (189.8, -50.0)
- added MX141: RShift, MX_Only:MXOnly-1.75U-Hotswap, F.Cu at (225.5, 31.0)
- added MX142: Up, MX_Only:MXOnly-1U-NoLED, F.Cu at (256.4, 35.7)
- added MX144: End, MX_Only:MXOnly-1U-NoLED, F.Cu at (280.3, 31.0)
- added MX162: RSpace, MX_Only:MXOnly-3U-ReversedStabilizers-NoLED, F.Cu at (137.4, 50.0)
- added MX164: RAlt, MX_Only:MXOnly-1U-NoLED, F.Cu at (175.5, 50.0)
- added MX167: RSuper, MX_Only:MXOnly-1U-Hotswap, F.Cu at (194.6, 50.0)
- added MX168: RCtrl, MX_Only:MXOnly-1U-NoLED, F.Cu at (213.6, 50.0)
- added MX17: F11, MX_Only:MXOnly-1U-Hotswap, F.Cu at (208.9, -50.0)
- added MX171: Left, MX_Only:MXOnly-1U-Hotswap, F.Cu at (237.4, 54.8)
- added MX173: Down, MX_Only:MXOnly-1U-Hotswap, F.Cu at (256.4, 54.8)
- added MX174: Right, MX_Only:MXOnly-1U-NoLED, F.Cu at (275.5, 54.8)
- added MX18: F12, MX_Only:MXOnly-1U-NoLED, F.Cu at (227.9, -50.0)
- added MX20: Pause, MX_Only:MXOnly-1U-NoLED, F.Cu at (251.7, -50.0)
- added MX23: Delete, MX_Only:MXOnly-1U-Hotswap, F.Cu at (280.3, -50.0)
- added MX38: 7, MX_Only:MXOnly-1U-NoLED, F.Cu at (118.4, -26.2)
- added MX40: 8, MX_Only:MXOnly-1U-NoLED, F.Cu at (137.4, -26.2)
- added MX42: 9, MX_Only:MXOnly-1U-NoLED, F.Cu at (156.5, -26.2)
- added MX44: 0, MX_Only:MXOnly-1U-NoLED, F.Cu at (175.5, -26.2)
- added MX47: -, MX_Only:MXOnly-1U-Hotswap, F.Cu at (194.6, -26.2)
- added MX49: =, MX_Only:MXOnly-1U-Hotswap, F.Cu at (213.6, -26.2)
- added MX51: Backspace, MX_Only:MXOnly-2U-NoLED, F.Cu at (242.2, -26.2)
- added MX54: Home, MX_Only:MXOnly-1U-NoLED, F.Cu at (280.3, -26.2)
- added MX63: Y, MX_Only:MXOnly-1U-NoLED, F.Cu at (108.8, -7.11)
- added MX66: U, MX_Only:MXOnly-1U-Hotswap, F.Cu at (127.9, -7.11)
- added MX68: I, MX_Only:MXOnly-1U-Hotswap, F.Cu at (146.9, -7.11)
- added MX69: O, MX_Only:MXOnly-1U-NoLED, F.Cu at (166.0, -7.11)
- added MX71: P, MX_Only:MXOnly-1U-NoLED, F.Cu at (185.0, -7.11)
- added MX74: [, MX_Only:MXOnly-1U-Hotswap, F.Cu at (204.1, -7.11)
- added MX75: ], MX_Only:MXOnly-1U-NoLED, F.Cu at (223.1, -7.11)
- added MX78: \, MX_Only:MXOnly-1.5U-Hotswap, F.Cu at (247.0, -7.11)
- added MX79: Pg Up, MX_Only:MXOnly-1U-NoLED, F.Cu at (280.3, -7.11)
- added MX9: F7, MX_Only:MXOnly-1U-Hotswap, F.Cu at (127.9, -50.0)
- added MX98: H, MX_Only:MXOnly-1U-Hotswap, F.Cu at (113.6, 11.9)
- added MX99: J, MX_Only:MXOnly-1U-NoLED, F.Cu at (132.7, 11.9)
- added R1: 5.1k, Footprints:R_0805_2012Metric, B.Cu at (278.5, -143.2)
- added R10: 10k, Footprints:R_0805_2012Metric, B.Cu at (278.8, -140.3)
- added R2: 5.1k, Footprints:R_0805_2012Metric, B.Cu at (270.0, -149.1)
- added R3: 5.1k, Footprints:R_0805_2012Metric, B.Cu at (274.4, -149.1)
- added R4: 5.1k, Footprints:R_0805_2012Metric, B.Cu at (282.9, -146.2)
- added R5: 10k, Footprints:R_0805_2012Metric, B.Cu at (287.6, -139.4)
- added R6: 10k, Footprints:R_0805_2012Metric, B.Cu at (283.2, -137.3)
- added R7: 22, Footprints:R_0805_2012Metric, B.Cu at (292.0, -139.4)
- added R8: 22, Footprints:R_0805_2012Metric, B.Cu at (353.7, -198.8)
- added R9: 10k, Footprints:R_0805_2012Metric, B.Cu at (287.3, -146.2)
- added USB1: HRO-TYPE-C-31-M-12, Footprints:HRO-TYPE-C-31-M-12, B.Cu at (261.2, -140.9)
- added USB2: HRO-TYPE-C-31-M-12, Footprints:HRO-TYPE-C-31-M-12, B.Cu at (294.8, -141.7)
- added Y1: Crystal_GND24_Small, Footprints:Crystal_SMD_3225-4Pin_3.2x2.5mm_HandSoldering, B.Cu at (-59.9, -32.9)
- added Y2: Crystal_GND24_Small, Footprints:Crystal_SMD_3225-4Pin_3.2x2.5mm_HandSoldering, B.Cu at (345.9, -209.0)
- D17, D83: moved to B.Cu
- MX100: renamed from MX73; footprint MX_Only:MXOnly-1U-NoLED -> MX_Only:MXOnly-1U-Hotswap
- MX102: renamed from MX74; footprint MX_Only:MXOnly-1U-NoLED -> MX_Only:MXOnly-1U-Hotswap
- MX104: renamed from MX75; footprint MX_Only:MXOnly-1U-NoLED -> MX_Only:MXOnly-1U-Hotswap
- MX106: renamed from MX76; footprint MX_Only:MXOnly-1U-NoLED -> MX_Only:MXOnly-1U-Hotswap
- MX112: renamed from MX79; footprint MX_Only:MXOnly-1U-NoLED -> MX_Only:MXOnly-1U-Hotswap
- MX131: renamed from MX97; footprint MX_Only:MXOnly-1U-NoLED -> MX_Only:MXOnly-1U-Hotswap
- MX135: renamed from MX99; footprint MX_Only:MXOnly-1U-NoLED -> MX_Only:MXOnly-1U-Hotswap
- MX143: renamed from MX103; footprint MX_Only:MXOnly-1U-NoLED -> MX_Only:MXOnly-1U-Hotswap
- MX145: renamed from MX104; footprint MX_Only:MXOnly-1U-NoLED -> MX_Only:MXOnly-1U-Hotswap
- MX15: renamed from MX16; footprint MX_Only:MXOnly-1U-NoLED -> MX_Only:MXOnly-1U-Hotswap
- MX163: renamed from MX121; footprint MX_Only:MXOnly-3U-ReversedStabilizers-NoLED -> MX_Only:MXOnly-1U-Hotswap
- MX165: renamed from MX122; footprint MX_Only:MXOnly-1U-NoLED -> MX_Only:MXOnly-1U-Hotswap
- MX169: renamed from MX124; footprint MX_Only:MXOnly-1U-NoLED -> MX_Only:MXOnly-1U-Hotswap
- MX175: renamed from MX127; footprint MX_Only:MXOnly-1U-NoLED -> MX_Only:MXOnly-1U-Hotswap
- MX19: renamed from MX18; footprint MX_Only:MXOnly-1U-NoLED -> MX_Only:MXOnly-1U-Hotswap
- MX21: renamed from MX19; footprint MX_Only:MXOnly-1U-NoLED -> MX_Only:MXOnly-1U-Hotswap
- MX39: renamed from MX37; footprint MX_Only:MXOnly-1U-NoLED -> MX_Only:MXOnly-1U-Hotswap
- MX41: renamed from MX38; footprint MX_Only:MXOnly-1U-NoLED -> MX_Only:MXOnly-1U-Hotswap
- MX43: renamed from MX39; footprint MX_Only:MXOnly-1U-NoLED -> MX_Only:MXOnly-1U-Hotswap
- MX45: renamed from MX40; footprint MX_Only:MXOnly-1U-NoLED -> MX_Only:MXOnly-1U-Hotswap
- MX52: renamed from MX45; footprint MX_Only:MXOnly-2U-NoLED -> MX_Only:MXOnly-2U-Hotswap
- MX55: renamed from MX46; footprint MX_Only:MXOnly-1U-NoLED -> MX_Only:MXOnly-1U-Hotswap
- MX64: renamed from MX47; footprint MX_Only:MXOnly-1U-NoLED -> MX_Only:MXOnly-1U-Hotswap
- MX70: renamed from MX50; footprint MX_Only:MXOnly-1U-NoLED -> MX_Only:MXOnly-1U-Hotswap
- MX72: renamed from MX51; footprint MX_Only:MXOnly-1U-NoLED -> MX_Only:MXOnly-1U-Hotswap
- MX76: renamed from MX53; footprint MX_Only:MXOnly-1U-NoLED -> MX_Only:MXOnly-1U-Hotswap
- MX80: renamed from MX55; footprint MX_Only:MXOnly-1U-NoLED -> MX_Only:MXOnly-1U-Hotswap
- U1, U2: footprint Package_QFP:TQFP-44_10x10mm_P0.8mm -> Footprints:QFN_TQFP-44_Combined; moved to B.Cu
- moved D87 399.6 mm to (223.6, 56.0)
- moved MX163 390.7 mm to (137.4, 50.0), turned to 180 degrees
- moved D41 389.1 mm to (257.0, -0.11)
- moved MX172 381.8 mm to (256.4, 54.8)
- moved MX140 377.6 mm to (225.5, 31.0)
- moved MX175 371.2 mm to (275.5, 54.8), turned to 180 degrees
- moved MX143 371.0 mm to (256.4, 35.7), turned to 180 degrees
- moved D90 360.0 mm to (282.5, 61.3)
- moved D57 356.8 mm to (246.8, 18.9)
- moved D58 339.1 mm to (287.3, 18.9)
- moved D42 334.0 mm to (287.3, -0.11)
- moved D71 333.0 mm to (209.3, 38.0)
- moved D15 333.0 mm to (287.3, -43.0)
- moved MX170 332.9 mm to (237.4, 54.8)
- moved MX166 327.0 mm to (194.6, 50.0)
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- renumbered MX14 to MX10, MX77 to MX107, MX78 to MX109, MX80 to MX113, MX82 to MX114, MX84 to MX115, MX86 to MX116, MX87 to MX117, MX89 to MX118, MX91 to MX119, MX15 to MX12, MX93 to MX120, MX95 to MX121, MX81 to MX122, MX83 to MX123, MX85 to MX124, MX88 to MX125, MX90 to MX126, MX92 to MX127, MX94 to MX128, MX96 to MX129, MX98 to MX132, MX100 to MX136, MX101 to MX138, MX102 to MX140, MX105 to MX146, MX107 to MX147, MX109 to MX148, MX111 to MX149, MX113 to MX150, MX115 to MX151, MX117 to MX152, MX119 to MX153, MX106 to MX154, MX108 to MX155, MX110 to MX156, MX112 to MX157, MX114 to MX158, MX116 to MX159, MX17 to MX16, MX118 to MX160, MX120 to MX161, MX123 to MX166, MX125 to MX170, MX126 to MX172, MX128 to MX176, MX130 to MX177, MX132 to MX178, MX134 to MX179, MX136 to MX180, MX138 to MX181, MX129 to MX182, MX131 to MX183, MX133 to MX184, MX135 to MX185, MX137 to MX186, MX139 to MX187, MX20 to MX22, MX21 to MX24, MX22 to MX25, MX4 to MX26, MX6 to MX27, MX8 to MX28, MX10 to MX29, MX12 to MX30, MX23 to MX31, MX25 to MX32, MX27 to MX33, MX29 to MX34, MX31 to MX35, MX33 to MX36, MX35 to MX37, MX5 to MX4, MX41 to MX46, MX42 to MX48, MX7 to MX5, MX24 to MX56, MX26 to MX57, MX28 to MX58, MX30 to MX59, MX9 to MX6, MX32 to MX60, MX34 to MX61, MX36 to MX62, MX48 to MX65, MX49 to MX67, MX11 to MX7, MX52 to MX73, MX54 to MX77, MX13 to MX8, MX57 to MX81, MX59 to MX82, MX61 to MX83, MX62 to MX84, MX64 to MX85, MX66 to MX86, MX68 to MX87, MX70 to MX88, MX56 to MX89, MX58 to MX90, MX60 to MX91, MX63 to MX92, MX65 to MX93, MX67 to MX94, MX69 to MX95, MX71 to MX96, MX72 to MX97
Connections:
- MX100 pad 1: CR2 -> Net-(D52-Pad2)
- MX100 pad 2: Net-(D52-Pad2) -> CR2
- MX102 pad 1: CR3 -> Net-(D53-Pad2)
- MX102 pad 2: Net-(D53-Pad2) -> CR3
- MX104 pad 1: CR4 -> Net-(D54-Pad2)
- MX104 pad 2: Net-(D54-Pad2) -> CR4
- MX106 pad 1: CR5 -> Net-(D55-Pad2)
- MX106 pad 2: Net-(D55-Pad2) -> CR5
- MX112 pad 1: CR8 -> Net-(D58-Pad2)
- MX112 pad 2: Net-(D58-Pad2) -> CR8
- MX131 pad 1: CR0 -> Net-(D67-Pad2)
- MX131 pad 2: Net-(D67-Pad2) -> CR0
- MX135 pad 1: CR3 -> Net-(D69-Pad2)
- MX135 pad 2: Net-(D69-Pad2) -> CR3
- MX143 pad 1: CR7 -> Net-(D73-Pad2)
- MX143 pad 2: Net-(D73-Pad2) -> CR7
- MX145 pad 1: CR8 -> Net-(D74-Pad2)
- MX145 pad 2: Net-(D74-Pad2) -> CR8
- MX15 pad 1: CR4 -> Net-(D11-Pad2)
- MX15 pad 2: Net-(D11-Pad2) -> CR4
- MX163 pad 1: CR0 -> Net-(D84-Pad2)
- MX163 pad 2: Net-(D84-Pad2) -> CR0
- MX165 pad 1: CR3 -> Net-(D85-Pad2)
- MX165 pad 2: Net-(D85-Pad2) -> CR3
- MX169 pad 1: CR5 -> Net-(D87-Pad2)
- MX169 pad 2: Net-(D87-Pad2) -> CR5
- MX175 pad 1: CR8 -> Net-(D90-Pad2)
- MX175 pad 2: Net-(D90-Pad2) -> CR8
- MX19 pad 1: CR6 -> Net-(D13-Pad2)
- MX19 pad 2: Net-(D13-Pad2) -> CR6
- MX21 pad 1: CR7 -> Net-(D14-Pad2)
- MX21 pad 2: Net-(D14-Pad2) -> CR7
- MX39 pad 1: CR0 -> Net-(D25-Pad2)
- MX39 pad 2: Net-(D25-Pad2) -> CR0
- MX41 pad 1: CR1 -> Net-(D26-Pad2)
- MX41 pad 2: Net-(D26-Pad2) -> CR1
- MX43 pad 1: CR2 -> Net-(D27-Pad2)
- MX43 pad 2: Net-(D27-Pad2) -> CR2
- MX45 pad 1: CR3 -> Net-(D28-Pad2)
- MX45 pad 2: Net-(D28-Pad2) -> CR3
- MX52 pad 1: CR7 -> Net-(D32-Pad2)
- MX52 pad 2: Net-(D32-Pad2) -> CR7
- MX55 pad 1: CR8 -> Net-(D33-Pad2)
- MX55 pad 2: Net-(D33-Pad2) -> CR8
- MX64 pad 1: CR0 -> Net-(D34-Pad2)
- MX64 pad 2: Net-(D34-Pad2) -> CR0
- MX70 pad 1: CR3 -> Net-(D37-Pad2)
- MX70 pad 2: Net-(D37-Pad2) -> CR3
- MX72 pad 1: CR4 -> Net-(D38-Pad2)
- MX72 pad 2: Net-(D38-Pad2) -> CR4
- MX76 pad 1: CR6 -> Net-(D40-Pad2)
- MX76 pad 2: Net-(D40-Pad2) -> CR6
- MX80 pad 1: CR8 -> Net-(D42-Pad2)
- MX80 pad 2: Net-(D42-Pad2) -> CR8
- U1 pad 14: Net-(U1-Pad14) -> +5V
- U1 pad 24: Net-(U1-Pad14) -> +5V
- U1 pad 34: Net-(U1-Pad14) -> +5V
- U1 pad 44: Net-(U1-Pad14) -> +5V
- U2 pad 14: Net-(U2-Pad14) -> +5VA
- U2 pad 24: Net-(U2-Pad14) -> +5VA
- U2 pad 34: Net-(U2-Pad14) -> +5VA
- U2 pad 44: Net-(U2-Pad14) -> +5VA
Routing:
- net RR2: track 0.00 -> 169.3 mm
- net RR3: track 0.00 -> 167.2 mm
- net RR1: track 0.00 -> 162.6 mm
- net RR4: track 0.00 -> 158.5 mm
- net RR0: track 0.00 -> 149.4 mm
- net CR6: track 0.00 -> 148.7 mm, vias 0 -> 4
- net CR7: track 0.00 -> 144.6 mm, vias 0 -> 5
- net CR5: track 0.00 -> 141.6 mm, vias 0 -> 5
- net CR4: track 0.00 -> 141.3 mm, vias 0 -> 5
- net CR3: track 0.00 -> 141.2 mm, vias 0 -> 5
- net RR5: track 0.00 -> 139.1 mm
- net CR8: track 0.00 -> 122.0 mm, vias 0 -> 5
- net CR2: track 0.00 -> 112.8 mm, vias 0 -> 4
- net CR0: track 0.00 -> 112.1 mm
- net CR1: track 0.00 -> 61.0 mm, vias 0 -> 1
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